File: schematic/car.kicad_pcb (KiCad board)
At the start: 2 copper layers, 3 parts

Commit message: Add JoystickReader.h here
Parts:
- added BTN: PushButton_6_pin, Connector_PinHeader_2.54mm:PushButton_6_pin, F.Cu at (61.0, 15.2)
- added POWERS: POWERS, Connector_PinHeader_2.54mm:PinHeader_2x03_P2.54mm_Vertical, F.Cu at (73.3, 20.7)
- added REF**: OUTPUTS, Connector_PinHeader_2.54mm:PinHeader_2x05_P2.54mm_Vertical, F.Cu at (73.5, 28.8)
Routing:
- net (no net): track 269.8 -> 539.6 mm, vias 4 -> 8
