File: schematic/remote/remote-big-good.kicad_pcb (KiCad board)
At the start: 2 copper layers, 16 parts, among them J2 Joystick_Right, J3 Joystick_Left, J4 Power-IN, U1 ARDUINO_PRO_MINI, U2 NRF24L01

Commit message: v2
Parts:
- removed the ? at (119.4, 17.8)
- removed the ? at (111.1, 17.8)
- removed the ? at (82.6, 38.7)
- removed the ? at (37.5, 25.4)
- removed the ? at (82.5, 23.6)
- removed the ? at (37.5, 17.1)
- removed the J4 at (16.5, 17.1)
- added ?: , , F.Cu at (92.4, 99.6)
- added ?: , , F.Cu at (92.4, 84.4)
- BTN: value PushButton -> PushButton_6_pin
- J2: value Joystick_Right -> Joystick_Left
- J3: value Joystick_Left -> Joystick_Right
- J4: value Power-IN -> Micro-Power-IN
- U2: value NRF24L01 -> NRF24L01_Breakout
- moved ? 63.9 mm to (113.4, 90.7)
- moved ? 63.9 mm to (43.2, 102.1)
- moved ? 63.9 mm to (123.5, 90.7)
- moved J4 63.9 mm to (40.6, 92.1)
- moved U1 63.9 mm to (110.8, 94.5)
- moved BTN 63.6 mm to (33.1, 103.3)
- moved U2 49.8 mm to (74.6, 79.4)
- moved J3 20.4 mm to (31.4, 37.5), turned to 90 degrees
- moved J2 19.7 mm to (103.2, 36.9), turned to 90 degrees
Connections:
- U1 pad JP6_5: Net-(J2-Pad2) -> Net-(J2-Pad3)
- U1 pad JP6_6: Net-(J2-Pad3) -> Net-(J2-Pad2)
- U1 pad JP6_7: Net-(J3-Pad3) -> Net-(J3-Pad2)
- U1 pad JP6_8: Net-(J3-Pad2) -> Net-(J3-Pad3)
Routing:
- net GND: track 267.2 -> 397.7 mm
- net +5V: track 249.6 -> 357.4 mm
- net Net-(J3-Pad2): track 80.1 -> 138.7 mm
- net Net-(J3-Pad1): track 76.4 -> 134.9 mm
- net Net-(J2-Pad1): track 52.9 -> 108.4 mm
- net Net-(J2-Pad2): track 6.03 -> 52.3 mm
- net Net-(J2-Pad3): track 6.03 -> 52.1 mm
- net Net-(J3-Pad3): track 87.9 -> 128.3 mm
- net Net-(U1-PadJP6_9): track 26.8 -> 35.8 mm
- net Net-(U1-PadJP6_10): track 35.2 -> 42.6 mm
- net Net-(U1-PadJP7_2): track 32.2 -> 38.4 mm
- net Net-(U1-PadJP6_11): track 27.8 -> 33.7 mm
- net Net-(U1-PadJP6_12): track 18.6 -> 23.8 mm
Other:
- board text removed: "+ -"
