File: schematic/remote/remote-small-good.kicad_pcb (KiCad board)
At the start: 2 copper layers, 16 parts, among them J2 Joystick_Right, J3 Joystick_Left, J4 Power-IN, U1 ARDUINO_PRO_MINI, U2 NRF24L01

Commit message: v2
Parts:
- removed the ? at (119.4, 17.8)
- removed the ? at (111.1, 17.8)
- removed the ? at (82.6, 38.7)
- removed the ? at (37.5, 25.4)
- removed the ? at (82.5, 23.6)
- removed the ? at (37.5, 17.1)
- removed the J4 at (16.5, 17.1)
- added ?: , , F.Cu at (94.0, 99.7)
- added ?: , , F.Cu at (119.4, 78.7)
- added ?: , , F.Cu at (128.9, 78.7)
- added ?: , , F.Cu at (94.0, 84.5)
- BTN: value PushButton -> PushButton_6_pin
- J2: value Joystick_Right -> Joystick_Left
- J3: value Joystick_Left -> Joystick_Right
- J4: value Power-IN -> Micro-Power-IN
- U2: value NRF24L01 -> NRF24L01_Breakout
- moved ? 64.2 mm to (114.9, 90.8)
- moved ? 64.2 mm to (125.1, 90.8)
- moved U1 64.2 mm to (112.4, 94.6)
- moved ? 63.8 mm to (55.9, 99.3)
- moved J4 63.8 mm to (53.3, 89.3)
- moved J3 62.0 mm to (45.1, 78.1)
- moved BTN 61.9 mm to (34.6, 101.3)
- moved J2 61.4 mm to (115.6, 78.7)
- moved U2 37.7 mm to (74.3, 67.3)
Connections:
- U1 pad JP6_7: Net-(J3-Pad3) -> Net-(J3-Pad2)
- U1 pad JP6_8: Net-(J3-Pad2) -> Net-(J3-Pad3)
Routing:
- net GND: track 267.2 -> 315.9 mm
- net Net-(U1-PadJP6_10): track 35.2 -> 71.1 mm
- net Net-(U1-PadJP6_11): track 27.8 -> 52.2 mm
- net Net-(U1-PadJP6_12): track 18.6 -> 42.2 mm
- net Net-(U1-PadJP7_2): track 32.2 -> 51.4 mm
- net Net-(U1-PadJP6_9): track 26.8 -> 45.6 mm
- net +5V: track 249.6 -> 263.3 mm
- net Net-(J3-Pad2): track 80.1 -> 92.2 mm
- net Net-(J2-Pad1): track 52.9 -> 58.0 mm
- net Net-(J3-Pad3): track 87.9 -> 92.4 mm
- net Net-(J2-Pad3): track 6.03 -> 9.04 mm
- net Net-(J2-Pad2): track 6.03 -> 9.04 mm
- net Net-(J3-Pad1): track 76.4 -> 77.9 mm
Other:
- board text removed: "+ -"
