File: schematic/remote/remote_bf.kicad_pcb (KiCad board)
At the start: 2 copper layers, 16 parts, among them J2 Joystick_Right, J3 Joystick_Left, J4 Power-IN, U1 ARDUINO_PRO_MINI, U2 NRF24L01

Commit message: v2
Parts:
- removed the ? at (106.4, 27.2)
- removed the ? at (119.4, 17.8)
- removed the ? at (111.1, 17.8)
- removed the ? at (116.5, 27.2)
- removed the ? at (82.6, 38.7)
- removed the ? at (37.5, 25.4)
- removed the ? at (82.5, 23.6)
- removed the ? at (37.5, 17.1)
- removed the J4 at (16.5, 17.1)
- added ?: , , F.Cu at (74.9, 89.5)
- added ?: , , F.Cu at (74.9, 100.3)
- added ?: , , F.Cu at (55.9, 31.1)
- added ?: , , F.Cu at (74.9, 83.2)
- added ?: , , F.Cu at (83.2, 31.8)
- added ?: , , F.Cu at (74.9, 87.0)
- added ?: , , F.Cu at (208.3, 62.9)
- added ?: , , F.Cu at (55.9, 22.2)
- added ?: , , F.Cu at (74.9, 97.2)
- added ?: , , F.Cu at (208.3, 52.1)
- added ?: , , F.Cu at (74.9, 76.8)
- added ?: , , F.Cu at (83.2, 24.8)
- added ?: , , F.Cu at (55.9, 62.2)
- added ?: , , F.Cu at (74.9, 80.6)
- added ?: , , F.Cu at (208.3, 39.4)
- added ?: , , F.Cu at (208.3, 43.2)
- added ?: , , F.Cu at (208.3, 59.7)
- added ?: , , F.Cu at (208.3, 45.7)
- added ?: , , F.Cu at (55.9, 72.4)
- added ?: , , F.Cu at (208.3, 49.5)
- BTN: value PushButton -> PushButton_6_pin
- J2: value Joystick_Right -> Joystick_Left
- J3: value Joystick_Left -> Joystick_Right
- U2: value NRF24L01 -> NRF24L01_Breakout
- moved U2 129.8 mm to (199.1, 41.8)
- moved ? 63.8 mm to (55.9, 99.3)
- moved J4 63.8 mm to (53.3, 89.3)
- moved BTN 61.9 mm to (34.6, 101.3)
- moved U1 61.7 mm to (109.2, 92.5)
- moved J2 5.85 mm to (104.1, 22.2), turned to 90 degrees
- moved J3 5.08 mm to (33.7, 22.2), turned to 90 degrees
Connections:
- U1 pad JP6_5: Net-(J2-Pad2) -> Net-(J2-Pad3)
- U1 pad JP6_6: Net-(J2-Pad3) -> Net-(J2-Pad2)
- U1 pad JP7_3: Net-(J3-Pad1) -> Net-(J2-Pad1)
- U1 pad JP7_4: Net-(J2-Pad1) -> Net-(J3-Pad1)
Routing:
- net GND: track 267.2 -> 411.0 mm
- net +5V: track 249.6 -> 364.3 mm
- net Net-(J2-Pad1): track 52.9 -> 127.6 mm
- net Net-(J2-Pad3): track 6.03 -> 63.7 mm
- net Net-(J2-Pad2): track 6.03 -> 63.7 mm
- net Net-(J3-Pad1): track 76.4 -> 130.7 mm
- net Net-(J3-Pad2): track 80.1 -> 123.5 mm
- net Net-(J3-Pad3): track 87.9 -> 124.0 mm
- net Net-(U1-PadJP7_2): track 32.2 -> 4.34 mm
- net Net-(U1-PadJP6_9): track 26.8 -> 14.5 mm
- net Net-(U1-PadJP6_10): track 35.2 -> 23.8 mm
- net Net-(U1-PadJP6_11): track 27.8 -> 19.5 mm
- net Net-(U1-PadJP6_12): track 18.6 -> 10.7 mm
Other:
- board text removed: "+ -"
