File: schematic/remote/remote-v1.kicad_pcb (KiCad board)
At the start: 2 copper layers, 13 parts, among them J2 Joystick_Left, J3 Joystick_Right, J4 Micro-Power-IN, J4 Power-IN, U2 NRF24L01_Breakout

Commit message: Works
Parts:
- removed the ? at (66.0, 30.5)
- removed the ? at (81.3, 25.4)
- removed the ? at (68.6, 30.5)
- removed A1: Arduino_Pro_Mini_Socket_NoSPH, PCM_arduino-library:Arduino_Pro_Mini_Socket_NoSPH
- added ?: , , F.Cu at (106.4, 27.2)
- added ?: , , F.Cu at (119.4, 17.8)
- added ?: , , F.Cu at (111.1, 17.8)
- added ?: , , F.Cu at (116.5, 27.2)
- added ?: , , F.Cu at (82.6, 38.7)
- added ?: , , F.Cu at (82.5, 23.6)
- added U1: ARDUINO_PRO_MINI, Arduino pro mini:MODULE_ARDUINO_PRO_MINI, B.Cu at (103.8, 31.0)
- J2: value Joystick_Left -> Joystick_Right
- J3: value Joystick_Right -> Joystick_Left
- J4: value Micro-Power-IN -> Power-IN
- U2: value NRF24L01_Breakout -> NRF24L01
- moved J3 43.3 mm to (33.7, 17.1)
- moved J2 35.2 mm to (107.9, 17.8)
- moved U2 31.5 mm to (69.9, 29.8)
Connections:
- J2 pad 1: JOYSTICK_LEFT_SW -> Net-(J2-Pad1)
- J2 pad 2: JOYSTICK_LEFT_Y -> Net-(J2-Pad2)
- J2 pad 3: JOYSTICK_LEFT_X -> Net-(J2-Pad3)
- J3 pad 1: JOYSTICK_RIGHT_SW -> Net-(J3-Pad1)
- J3 pad 2: JOYSTICK_RIGHT_Y -> Net-(J3-Pad2)
- J3 pad 3: JOYSTICK_RIGHT_X -> Net-(J3-Pad3)
- U2 pad 3: NRF_CE -> Net-(U1-PadJP7_2)
- U2 pad 4: NRF_CSN -> Net-(U1-PadJP6_12)
- U2 pad 5: NRF_SCK -> Net-(U1-PadJP6_9)
- U2 pad 6: NRF_MOSI -> Net-(U1-PadJP6_11)
- U2 pad 7: NRF_MISO -> Net-(U1-PadJP6_10)
Routing:
- net GND: track 175.4 -> 267.2 mm
- net Net-(J3-Pad3): track 0.00 -> 87.9 mm
- net Net-(J3-Pad2): track 0.00 -> 80.1 mm
- net +5V: track 176.2 -> 249.6 mm
- net Net-(J3-Pad1): track 8.26 -> 76.4 mm
- net Net-(J2-Pad1): track 0.00 -> 52.9 mm
- net NRF_SCK: track 38.1 -> 0.00 mm
- net Net-(U1-PadJP6_10): track 0.00 -> 35.2 mm
- net Net-(U1-PadJP7_2): track 0.00 -> 32.2 mm
- net NRF_CSN: track 27.9 -> 0.00 mm
- net NRF_CE: track 27.9 -> 0.00 mm
- net Net-(U1-PadJP6_11): track 0.00 -> 27.8 mm
- net Net-(U1-PadJP6_9): track 0.00 -> 26.8 mm
- net NRF_MISO: track 25.4 -> 0.00 mm
- net NRF_MOSI: track 25.4 -> 0.00 mm
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Other:
- board text removed: "+"
- board text removed: "-"
- board text removed: "- +"
- board text removed: "8V->5v"
- board text removed: "A"
- board text removed: "B"
- board text removed: "D"
- board text removed: "GND"
- board text removed: "Melorin Car"
- board text removed: "Motor"
- board text removed: "V5"
- board text removed: "VCC"
- board text removed: "^ ^"
