File: schematic/remote/remote.kicad_sch (KiCad schematic)
At the start: 6 parts, among them J1 Conn_01x05_Male, J2 Joystick_Left, J3 Joystick_Right, J4 Micro-Power-IN, J5 NRF-Power, U1 ARDUINO_PRO_MINI

Commit message: v2
Parts:
- removed J1: Conn_01x05_Male, Connector_PinHeader_2.54mm:PinHeader_1x05_P2.54mm_Vertical, symbol Connector:Conn_01x05_Male
- removed J5: NRF-Power, Connector_PinHeader_2.54mm:PinHeader_1x02_P2.54mm_Vertical, symbol Connector:Conn_01x02_Male
- added U2: NRF24L01_Breakout, Arduino pro mini:NRF24L01, symbol RF:NRF24L01_Breakout
Connections:
- net +5V: now also U2.2 (VCC)
- net GND: now also U2.1 (GND)
- net at U1.JP7_2 (D8): now also U2.3 (CE)
- net at U1.JP6_12 (D10): now also U2.4 (~{CSN})
- net at U1.JP6_9 (SCK): now also U2.5 (SCK)
- net at U1.JP6_10 (MISO): now also U2.7 (MISO)
- net at U1.JP6_11 (MOSI): now also U2.6 (MOSI)
- net at U1.JP6_5 (A3): now also J2.2 (Pin_2); no longer J3.2 (Pin_2)
- net at U1.JP6_6 (A2): now also J2.3 (Pin_3); no longer J3.3 (Pin_3)
- net at U1.JP6_7 (A1): now also J3.3 (Pin_3); no longer J2.2 (Pin_2)
- net at U1.JP6_8 (A0): now also J3.2 (Pin_2); no longer J2.3 (Pin_3)
- net at U1.JP7_3 (D7): now also J3.1 (Pin_1); no longer J2.1 (Pin_1)
- net at U1.JP7_4 (D6): now also J2.1 (Pin_1); no longer J3.1 (Pin_1)

Commit message: Works
Parts:
- removed U1: ARDUINO_PRO_MINI, MODULE_ARDUINO_PRO_MINI, symbol Arduino pro mini:ARDUINO_PRO_MINI
- added A1: Arduino_Pro_Mini_Socket_NoSPH, PCM_arduino-library:Arduino_Pro_Mini_Socket_NoSPH, symbol PCM_arduino-library:Arduino_Pro_Mini_Socket_NoSPH
Connections:
- net +5V: now also A1.Vcc1 (Vcc)
- net GND: now also A1.GND1 (GND), A1.GND2 (GND)
- net NRF_MISO: now reaches U2.7 (MISO)
- net NRF_MISO: now also A1.D12 (D12_MISO)
- net NRF_MOSI: now reaches U2.6 (MOSI)
- net NRF_MOSI: now also A1.D11 (D11_MOSI)
- net NRF_CSN: now reaches U2.4 (~{CSN})
- net NRF_CSN: now also A1.D10 (D10_CS)
- net JOYSTICK_LEFT_Y: now reaches J2.2 (Pin_2)
- net JOYSTICK_LEFT_Y: now also A1.A2
- net JOYSTICK_LEFT_X: now reaches J2.3 (Pin_3)
- net JOYSTICK_LEFT_X: now also A1.A3
- net JOYSTICK_RIGHT_X: now reaches J3.3 (Pin_3)
- net JOYSTICK_RIGHT_X: now also A1.A1
- net JOYSTICK_RIGHT_Y: now reaches J3.2 (Pin_2)
- net JOYSTICK_RIGHT_Y: now also A1.A0
- net NRF_SCK: now reaches U2.5 (SCK)
- net NRF_SCK: now also A1.D13 (D13_SCK)
- net NRF_CE: now reaches U2.3 (CE)
- net NRF_CE: now also A1.D8
- net JOYSTICK_RIGHT_SW: now reaches J3.1 (Pin_1)
- net JOYSTICK_RIGHT_SW: now also A1.D4
- net JOYSTICK_LEFT_SW: now reaches J2.1 (Pin_1)
- net JOYSTICK_LEFT_SW: now also A1.D5
Other:
- moved on the sheet: J4
