File: schematic/car/car_sch.kicad_pcb (KiCad board)
At the start: 2 copper layers, 18 parts, among them J1 Led, J10 Motor-PWR-IN, J2 Servo, J3 NRF-Power, J4 Accel, J5 Micro-Power-IN, J6 MOTOR-CTRL, J7 MOTOR-PWR-OUT, J8 Horn, U1 ARDUINO_PRO_MINI

Commit message: e
Parts:
- removed ? (x6): , 
- removed J10: Motor-PWR-IN, Connector_PinHeader_2.54mm:PinHeader_1x02_P2.54mm_Vertical
- BTN: value PushButton_6_pin -> Power_btn
- J1: value Led -> Led (D+-)
- J2: value Servo -> Servo (D+-); moved to F.Cu
- J3: value NRF-Power -> NRF_Power
- J8: value Horn -> Horn (+-)
- NRF1: value Conn_01x06_Male -> NRF24L01
- moved J7 21.0 mm to (111.8, 35.6)
- moved J4 9.53 mm to (83.2, 36.2)
- moved J8 9.44 mm to (83.2, 40.0)
- moved J1 8.98 mm to (88.2, 32.4)
- moved J5 8.18 mm to (97.8, 35.6)
- moved J3 7.34 mm to (36.8, 43.0)
- moved J6 7.10 mm to (83.2, 26.0)
- moved NRF1 6.95 mm to (24.4, 29.1)
- moved U1 6.95 mm to (60.0, 31.1)
- moved BTN 6.57 mm to (98.7, 20.6)
- moved J2 5.85 mm to (88.2, 18.4), turned to -90 degrees
Connections:
- BTN pad 4: +12V -> GND
- BTN pad 6: +12V -> GND
- J7 pad 1: +12V -> +5V
Routing:
- net +5V: track 180.7 -> 262.5 mm
- net Net-(J2-Pad3): track 111.1 -> 166.1 mm
- net GND: track 158.4 -> 204.3 mm
- net +12V: track 31.0 -> 0.00 mm
- net Net-(NRF1-Pad2): track 26.3 -> 48.2 mm
- net Net-(NRF1-Pad1): track 35.9 -> 50.3 mm
- net Net-(NRF1-Pad5): track 35.1 -> 42.3 mm
- net Net-(NRF1-Pad4): track 39.9 -> 44.1 mm
- net Net-(NRF1-Pad3): track 45.3 -> 49.5 mm
- net Net-(J1-Pad3): track 30.3 -> 34.2 mm
- net Net-(J4-Pad1): track 29.5 -> 27.6 mm
- net Net-(J8-Pad1): track 25.0 -> 24.1 mm
- net Net-(J6-Pad2): track 44.7 -> 44.1 mm
Other:
- board text added: "0"
- board text added: "5V"
- board text added: "<- 5V ->"
- board text added: "<- GND ->"
- board text added: "Arduino Pro Mini"
- board text added: "GND"

Commit message: v2
Parts:
- removed J3: NRF_Power, Connector_PinHeader_2.54mm:PinHeader_1x02_P2.54mm_Vertical
- removed NRF1: NRF24L01, Connector_PinHeader_2.54mm:PinHeader_1x06_P2.54mm_Vertical
- added J9: Powers, Connector_PinHeader_2.54mm:PinHeader_2x04_P2.54mm_Vertical, F.Cu at (49.8, 53.6)
- added U2: NRF24L01, Arduino pro mini:NRF24L01, F.Cu at (35.6, 26.7)
- moved J7 67.6 mm to (46.0, 51.0)
- moved BTN 51.2 mm to (72.0, 64.3), turned to 180 degrees
- moved J5 49.8 mm to (55.5, 61.8), turned to -90 degrees
- moved J2 31.6 mm to (72.4, 45.7)
- moved J8 22.0 mm to (67.3, 24.8)
- moved J6 21.1 mm to (67.3, 40.0)
- moved J4 17.1 mm to (67.3, 29.8)
- moved J1 16.1 mm to (72.4, 34.9)
- moved U1 5.22 mm to (54.8, 30.5), turned to 180 degrees
Connections:
- BTN pad 3: +5V -> GND
- BTN pad 4: GND -> +5V
- BTN pad 5: +5V -> GND
- BTN pad 6: GND -> +5V
Routing:
- net Net-(J2-Pad3): track 166.1 -> 4.87 mm
- net +5V: track 262.5 -> 180.0 mm
- net GND: track 204.3 -> 164.2 mm
- net Net-(J6-Pad1): track 44.4 -> 5.15 mm
- net Net-(J6-Pad2): track 44.1 -> 8.51 mm
- net Net-(J1-Pad3): track 34.2 -> 5.13 mm
- net Net-(U1-PadJP6_10): track 44.1 -> 16.2 mm
- net Net-(U1-PadJP6_9): track 49.5 -> 25.1 mm
- net Net-(J4-Pad1): track 27.6 -> 5.15 mm
- net Net-(U1-PadJP6_11): track 42.3 -> 20.4 mm
- net Net-(U1-PadJP6_12): track 48.2 -> 27.3 mm
- net Net-(J8-Pad1): track 24.1 -> 6.88 mm
- net Net-(U1-PadJP7_2): track 50.3 -> 49.1 mm
Other:
- board text added: "- +"
- board text added: "V2"
- board text removed: "0"
- board text removed: "5V"
- board text removed: "<- 5V ->"
- board text removed: "<- GND ->"
- board text removed: "GND"

Commit message: drv8833
Parts:
- removed BTN: Power_btn, Connector_PinHeader_2.54mm:PushButton_6_pin
- removed J4: Accel, Connector_PinHeader_2.54mm:PinHeader_1x01_P2.54mm_Vertical
- removed J7: MOTOR-PWR-OUT, Connector_PinHeader_2.54mm:PinHeader_1x02_P2.54mm_Vertical
- removed J9: Powers, Connector_PinHeader_2.54mm:PinHeader_2x04_P2.54mm_Vertical
- added A1: , PCM_arduino-library:Arduino_Pro_Mini_Socket_NoSPH, B.Cu at (45.7, 30.5)
- added J13: Regulator-9v, Connector_PinHeader_2.54mm:PinHeader_2x02_P2.54mm_Vertical, B.Cu at (71.1, 58.4)
- added J14: Input-Motor, Connector_PinHeader_2.54mm:PinHeader_1x02_P2.54mm_Vertical, B.Cu at (71.1, 61.0)
- added J16: Button, Connector_PinHeader_2.54mm:PinHeader_2x02_P2.54mm_Vertical, F.Cu at (68.6, 61.0)
- added J3: Input-Micro, Connector_PinHeader_2.54mm:PinHeader_1x02_P2.54mm_Vertical, F.Cu at (63.5, 61.0)
- J1: value Led (D+-) -> < Led
- J2: value Servo (D+-) -> < Servo
- J5: value Micro-Power-IN -> Regulator-5v; footprint Connector_PinHeader_2.54mm:PinHeader_1x02_P2.54mm_Vertical -> Connector_PinHeader_2.54mm:PinHeader_2x02_P2.54mm_Vertical
- J6: value MOTOR-CTRL -> Motor
- J8: value Horn (+-) -> Horn
- U1: value ARDUINO_PRO_MINI -> DRV8833; footprint Arduino pro mini:MODULE_ARDUINO_PRO_MINI -> Package_SO:TSSOP-16_4.4x5mm_P0.65mm; moved to F.Cu
- U2: value NRF24L01 -> NRF24L01_Breakout
- moved J8 17.1 mm to (61.0, 40.6)
- moved U1 14.7 mm to (68.6, 25.4), turned to -90 degrees
- moved J1 12.1 mm to (63.5, 43.2)
- moved U2 10.2 mm to (25.4, 26.7)
- moved J2 8.89 mm to (63.5, 45.7)
- moved J5 8.67 mm to (63.5, 58.4), turned to 180 degrees
- moved J6 3.85 mm to (71.1, 40.6), turned to -90 degrees
Connections:
- J1 pad 1: GND -> GND2
- J1 pad 3: Net-(J1-Pad3) -> PIN_LED
- J2 pad 1: GND -> GND2
- J2 pad 3: Net-(J2-Pad3) -> PIN_SERVO
- J5 pad 1: +5V -> Net-(J16-Pad4)
- J5 pad 2: GND -> Net-(J3-Pad2)
- J8 pad 1: Net-(J8-Pad1) -> PIN_HORN
- J8 pad 2: GND -> GND2
- U2 pad 1: GND -> GND2
- U2 pad 3: Net-(U1-PadJP7_2) -> NRF_CE
- U2 pad 4: Net-(U1-PadJP6_12) -> NRF_CSN
- U2 pad 5: Net-(U1-PadJP6_9) -> NRF_SCK
- U2 pad 6: Net-(U1-PadJP6_11) -> NRF_MOSI
- U2 pad 7: Net-(U1-PadJP6_10) -> NRF_MISO
Routing:
- net GND2: track 0.00 -> 175.8 mm
- net GND: track 164.2 -> 0.00 mm
- net +9V: track 0.00 -> 53.3 mm
- net GND1: track 0.00 -> 52.3 mm
- net NRF_CE: track 0.00 -> 50.2 mm
- net PIN_MOTOR_2: track 0.00 -> 49.7 mm
- net Net-(U1-PadJP7_2): track 49.1 -> 0.00 mm
- net PIN_MOTOR_1: track 0.00 -> 35.6 mm
- net NRF_CSN: track 0.00 -> 28.3 mm
- net Net-(U1-PadJP6_12): track 27.3 -> 0.00 mm
- net NRF_SCK: track 0.00 -> 26.2 mm
- net Net-(U1-PadJP6_9): track 25.1 -> 0.00 mm
- net NRF_MOSI: track 0.00 -> 21.4 mm
- net Net-(U1-PadJP6_11): track 20.4 -> 0.00 mm
- net +5V: track 180.0 -> 161.9 mm
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Other:
- board text added: "Melorin Car"

Commit message: schematic
Parts:
- removed A1: , PCM_arduino-library:Arduino_Pro_Mini_Socket_NoSPH
- removed J13: Regulator-9v, Connector_PinHeader_2.54mm:PinHeader_2x02_P2.54mm_Vertical
- removed J14: Input-Motor, Connector_PinHeader_2.54mm:PinHeader_1x02_P2.54mm_Vertical
- removed J16: Button, Connector_PinHeader_2.54mm:PinHeader_2x02_P2.54mm_Vertical
- added ?: , , F.Cu at (76.2, 40.6)
- added ?: , , F.Cu at (76.2, 45.7)
- added ?: , , F.Cu at (76.2, 50.8)
- added ?: , , F.Cu at (76.2, 55.9)
- added A3: Arduino_Pro_Mini_Socket_NoSPH, PCM_arduino-library:Arduino_Pro_Mini_Socket_NoSPH, B.Cu at (45.7, 33.0)
- added J4: Power, Connector_PinHeader_2.54mm:PinHeader_1x02_P2.54mm_Vertical, F.Cu at (68.6, 58.4)
- added J7: BarGraph, Connector_PinHeader_2.54mm:PinHeader_1x02_P2.54mm_Vertical, F.Cu at (55.9, 58.4)
- J1: value < Led -> Led
- J2: value < Servo -> Servo
- J3: value Input-Micro -> Battery
- J5: value Regulator-5v -> Switch
- J6: value Motor -> MOTOR-CTRL
- U1: value DRV8833 -> DRV8833PW
- moved J3 10.5 mm to (53.3, 58.4), turned to 180 degrees
- moved J6 2.54 mm to (68.6, 40.6), turned to 0 degrees
- moved U1 2.54 mm to (68.6, 27.9)
- moved J1 2.54 mm to (63.5, 45.7)
- moved J2 2.54 mm to (63.5, 48.3)
- moved J8 2.54 mm to (61.0, 43.2)
- moved U2 2.54 mm to (25.4, 29.2)
- turned J5 to 90 degrees
Connections:
- J1 pad 1: GND2 -> GND
- J2 pad 1: GND2 -> GND
- J3 pad 1: Net-(J16-Pad2) -> -BATT
- J3 pad 2: Net-(J3-Pad2) -> +BATT
- J5 pad 1: Net-(J16-Pad4) -> +8V
- J5 pad 2: Net-(J3-Pad2) -> +BATT
- J5 pad 3: +5V -> +8V
- J5 pad 4: GND2 -> +BATT
- J8 pad 2: GND2 -> GND
- U1 pad 11: +9V -> +8V
- U1 pad 13: GND1 -> GND
- U2 pad 1: GND2 -> GND
Routing:
- net GND2: track 175.8 -> 0.00 mm
- net +8V: track 0.00 -> 128.7 mm
- net GND: track 0.00 -> 97.8 mm
- net +5V: track 161.9 -> 106.5 mm
- net +9V: track 53.3 -> 0.00 mm
- net GND1: track 52.3 -> 0.00 mm
- net +BATT: track 0.00 -> 25.4 mm
- net Net-(J6-Pin_2): track 7.62 -> 22.9 mm
- net Net-(J6-Pin_1): track 7.62 -> 12.7 mm
- net NRF_CSN: track 28.3 -> 24.7 mm
- net Net-(J16-Pad4): track 2.54 -> 0.00 mm
- net Net-(J16-Pad2): track 2.54 -> 0.00 mm
- net Net-(J14-Pad1): track 2.54 -> 0.00 mm
- net Net-(J13-Pad1): track 2.54 -> 0.00 mm
- net Net-(J3-Pad2): track 2.54 -> 0.00 mm
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Other:
- board text added: "A"
- board text added: "B"
- board text added: "BAT"
- board text added: "GND"
- board text added: "PWR"
- board text added: "V4"
- board text added: "VCC"
- board text removed: "- +"
- board text removed: "Arduino Pro Mini"
- board text removed: "V2"

Commit message: wip
Parts:
- moved ? 29.0 mm to (94.0, 17.8)
- moved ? 29.0 mm to (94.0, 22.9)
- moved ? 29.0 mm to (94.0, 28.0)
- moved ? 29.0 mm to (94.0, 33.0)
- moved J4 22.7 mm to (88.9, 48.3)
- moved J7 22.7 mm to (76.2, 48.3)
- moved J3 22.7 mm to (73.7, 48.3)
- moved J5 22.7 mm to (83.8, 48.3)
- moved J6 16.3 mm to (81.3, 30.5)
Routing:
- net Net-(J6-Pin_1): track 12.7 -> 40.6 mm
- net GND: track 97.8 -> 123.2 mm
- net Net-(J6-Pin_2): track 22.9 -> 43.2 mm
- net +8V: track 128.7 -> 145.7 mm
Other:
- board text added: "+"
- board text added: "-"
- board text added: "D"
- board text added: "V5"
- board text removed: "V4"

Commit message: Works
Parts:
- removed the ? at (94.0, 28.0)
- removed the ? at (94.0, 33.0)
- removed J6: MOTOR-CTRL, Connector_PinHeader_2.54mm:PinHeader_1x02_P2.54mm_Vertical
- added ?: Extra, Connector_PinHeader_2.54mm:PinHeader_1x02_P2.54mm_Vertical, F.Cu at (58.4, 45.7)
- added ?: , , F.Cu at (55.9, 25.4)
- added ?: Reg-IN, Connector_PinHeader_2.54mm:PinHeader_1x02_P2.54mm_Vertical, F.Cu at (48.3, 22.9)
- added ?: Reg-OUT, Connector_PinHeader_2.54mm:PinHeader_1x02_P2.54mm_Vertical, F.Cu at (48.3, 20.3)
- added ?: Lamps, Connector_PinHeader_2.54mm:PinHeader_1x02_P2.54mm_Vertical, F.Cu at (58.4, 48.3)
- added ?: , , F.Cu at (61.0, 25.4)
- added JP1: Use regulator, Connector_PinHeader_2.54mm:PinHeader_1x02_P2.54mm_Vertical, F.Cu at (43.2, 35.6)
- ?: renamed from J7; moved to B.Cu
- ?: renamed from J3; moved to B.Cu
- A3: value Arduino_Pro_Mini_Socket_NoSPH -> Arduino Pro Mini
- J5: moved to B.Cu
- U1: value DRV8833PW -> DRV8833
- U2: value NRF24L01_Breakout -> NRF24L01
- moved ? 76.2 mm to (17.8, 20.3), turned to 90 degrees
- moved ? 71.2 mm to (22.9, 20.3), turned to 90 degrees
- moved U1 43.8 mm to (25.4, 35.6), turned to 180 degrees
- moved ? 33.1 mm to (61.0, 30.5), turned to -90 degrees
- moved J5 29.6 mm to (58.4, 33.0), turned to -90 degrees
- moved U2 22.9 mm to (25.7, 52.2)
- moved ? 19.3 mm to (58.4, 40.6), turned to 0 degrees
- moved A3 15.2 mm to (45.7, 48.3)
- moved ? 14.8 mm to (61.0, 40.6), turned to 0 degrees
- moved J1 13.0 mm to (61.0, 58.4)
- moved J2 13.0 mm to (61.0, 61.0)
- moved J8 8.03 mm to (58.4, 50.8)
- renumbered J4 to ?
Connections:
- A3 pad D2: unconnected-(A3-D2_INT0-PadD2) -> EXTRA
- A3 pad D3: unconnected-(A3-D3_INT1-PadD3) -> LAMPS
- A3 pad RAW: +8V -> Net-(JP1-B)
Routing:
- net +8V: track 145.7 -> 71.1 mm
- net +5V: track 106.5 -> 151.2 mm
- net Net-(J6-Pin_2): track 43.2 -> 20.3 mm
- net +BATT: track 25.4 -> 5.08 mm
- net Net-(J6-Pin_1): track 40.6 -> 22.9 mm
- net PIN_HORN: track 15.2 -> 5.08 mm
- net PIN_MOTOR_1: track 36.0 -> 45.7 mm
- net NRF_SCK: track 26.6 -> 17.8 mm
- net Net-(JP1-B): track 0.00 -> 7.62 mm
- net LAMPS: track 0.00 -> 5.08 mm
- net EXTRA: track 0.00 -> 5.08 mm
- net NRF_MISO: track 15.0 -> 10.2 mm
- net GND: track 123.2 -> 127.9 mm
- net NRF_MOSI: track 19.3 -> 15.2 mm
- net PIN_LED: track 6.13 -> 2.46 mm
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Other:
- board text added: "- +"
- board text added: "8V->5v"
- board text added: "Motor"
- board text added: "^ ^"
- board text removed: "BAT"
- board text removed: "MeloCar Engine"
- board text removed: "PWR"
