File: schematic/car/car_sch.kicad_sch (KiCad schematic)
At the start: 11 parts, among them J1 Led, J10 Motor-PWR-IN, J2 Servo, J3 NRF-Power, J4 Conn_01x01_Male, J5 Micro-Power-IN, J6 MOTOR-CTRL, J7 MOTOR-PWR-OUT, J8 Horn, U1 ARDUINO_PRO_MINI

Commit message: e
Parts:
- J4: value Conn_01x01_Male -> Accel
- NRF1: value Conn_01x06_Male -> NRF24L01
Connections:
- net +12V: no longer J7.1 (Pin_1)
- net +5V: now also J7.1 (Pin_1)
Changed lines of the file:
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@@
     (in_bom yes) (on_board yes) (fields_autoplaced)
     (property "Reference" "J4" (id 0) (at 89.535 53.34 0))
-    (property "Value" "Conn_01x01_Male" (id 1) (at 89.535 55.88 0))
+    (property "Value" "Accel" (id 1) (at 89.535 55.88 0))
     (property "Footprint" "Connector_PinHeader_2.54mm:PinHeader_1x01_P2.54mm_Vertical" (id 2) (at 88.9 58.42 0)
       (effects (font (size 1.27 1.27)) hide)
@@
     (pin "1")
   )
-  (symbol (lib_id "power:+12V") (at 91.44 76.2 270) (unit 1)
-    (in_bom yes) (on_board yes) (fields_autoplaced)
-    (property "Reference" "#PWR0113" (id 0) (at 87.63 76.2 0)
-      (effects (font (size 1.27 1.27)) hide)
-    )
-    (property "Value" "+12V" (id 1) (at 95.25 76.1999 90)
-      (effects (font (size 1.27 1.27)) (justify left))
-    )
-    (property "Footprint" "" (id 2) (at 91.44 76.2 0)
-      (effects (font (size 1.27 1.27)) hide)
-    )
-    (property "Datasheet" "" (id 3) (at 91.44 76.2 0)
-      (effects (font (size 1.27 1.27)) hide)
-    )
-    (pin "1")
-  )
   (symbol (lib_id "Connector:Conn_01x03_Male") (at 118.11 48.26 0) (unit 1)
     (in_bom yes) (on_board yes) (fields_autoplaced)
@@
       (effects (font (size 1.27 1.27)) (justify right))
     )
-    (property "Value" "Conn_01x06_Male" (id 1) (at 101.6 92.7099 0)
+    (property "Value" "NRF24L01" (id 1) (at 101.6 92.7099 0)
       (effects (font (size 1.27 1.27)) (justify right))
     )
@@
     (pin "2")
   )
+  (symbol (lib_id "power:+5V") (at 91.44 76.2 270) (unit 1)
+    (in_bom yes) (on_board yes) (fields_autoplaced)
+    (property "Reference" "#PWR0108" (id 0) (at 87.63 76.2 0)
+      (effects (font (size 1.27 1.27)) hide)
+    )
+    (property "Value" "+5V" (id 1) (at 95.25 76.1999 90)
+      (effects (font (size 1.27 1.27)) (justify left))
+    )
+    (property "Footprint" "" (id 2) (at 91.44 76.2 0)
+      (effects (font (size 1.27 1.27)) hide)
+    )
+    (property "Datasheet" "" (id 3) (at 91.44 76.2 0)
+      (effects (font (size 1.27 1.27)) hide)
+    )
+    (pin "1")
+  )
   (symbol (lib_id "power:GND") (at 124.46 59.69 90) (unit 1)
     (in_bom yes) (on_board yes) (fields_autoplaced)
@@
   (symbol (lib_id "power:GND") (at 26.67 63.5 270) (unit 1)
     (in_bom yes) (on_board yes) (fields_autoplaced)
-    (property "Reference" "#PWR?" (id 0) (at 20.32 63.5 0)
+    (property "Reference" "#PWR0107" (id 0) (at 20.32 63.5 0)
       (effects (font (size 1.27 1.27)) hide)
     )
@@
       (reference "#PWR0106") (unit 1) (value "GND") (footprint "")
     )
+    (path "/ff16ee3c-e788-484d-ae7a-18b27e86f391"
+      (reference "#PWR0107") (unit 1) (value "GND") (footprint "")
+    )
+    (path "/e19ee15a-d6dc-40bc-8daf-0b9ae8be0bdd"
+      (reference "#PWR0108") (unit 1) (value "+5V") (footprint "")
+    )
     (path "/3cdf2078-c986-49ab-882b-11f67003c171"
       (reference "#PWR0109") (unit 1) (value "GND") (footprint "")
@@
       (reference "#PWR0112") (unit 1) (value "+5V") (footprint "")
     )
-    (path "/5c05cc92-a085-4821-986d-1508f4b72961"
-      (reference "#PWR0113") (unit 1) (value "+12V") (footprint "")
-    )
     (path "/544893c4-81c4-4324-837c-56d6520110ab"
       (reference "#PWR0114") (unit 1) (value "GND") (footprint "")
@@
       (reference "#PWR0117") (unit 1) (value "GND") (footprint "")
     )
-    (path "/ff16ee3c-e788-484d-ae7a-18b27e86f391"
-      (reference "#PWR?") (unit 1) (value "GND") (footprint "")
-    )
     (path "/5f0cb4f5-99dd-431c-94d2-6151fa427b3a"
       (reference "J1") (unit 1) (value "Led") (footprint "Connector_PinHeader_2.54mm:PinHeader_1x03_P2.54mm_Vertical")
@@
     )
     (path "/462ba2d8-20cc-4820-b227-ba02d60db96d"
-      (reference "J4") (unit 1) (value "Conn_01x01_Male") (footprint "Connector_PinHeader_2.54mm:PinHeader_1x01_P2.54mm_Vertical")
+      (reference "J4") (unit 1) (value "Accel") (footprint "Connector_PinHeader_2.54mm:PinHeader_1x01_P2.54mm_Vertical")
     )
     (path "/489b3162-1756-4d9c-8b75-ba1ffece0b1e"
@@
     )
     (path "/bf74795d-5121-4722-b0f3-84275bd5c707"
-      (reference "NRF1") (unit 1) (value "Conn_01x06_Male") (footprint "Connector_PinHeader_2.54mm:PinHeader_1x06_P2.54mm_Vertical")
+      (reference "NRF1") (unit 1) (value "NRF24L01") (footprint "Connector_PinHeader_2.54mm:PinHeader_1x06_P2.54mm_Vertical")
     )
     (path "/1211422c-155d-4bd7-a798-21ca94f38c11"

Commit message: v2
Parts:
- removed NRF1: NRF24L01, Connector_PinHeader_2.54mm:PinHeader_1x06_P2.54mm_Vertical, symbol Connector:Conn_01x06_Male
- added J9: Powers, Connector_PinHeader_2.54mm:PinHeader_2x04_P2.54mm_Vertical, symbol Connector_Generic:Conn_02x04_Counter_Clockwise
- added U2: NRF24L01_Breakout, Arduino pro mini:NRF24L01, symbol RF:NRF24L01_Breakout
Connections:
- net +5V: now also U2.2 (VCC)
- net GND: now also U2.1 (GND)
- net at U1.JP6_10 (MISO): now also U2.7 (MISO)
- net at U1.JP6_11 (MOSI): now also U2.6 (MOSI)
- net at U1.JP6_12 (D10): now also U2.4 (~{CSN})
- net at U1.JP6_9 (SCK): now also U2.5 (SCK)
- net at U1.JP7_2 (D8): now also U2.3 (CE)

Commit message: drv8833
Parts:
- removed J10: Motor-PWR-IN, Connector_PinHeader_2.54mm:PinHeader_1x02_P2.54mm_Vertical, symbol Connector:Conn_01x02_Male
- removed J5: Micro-Power-IN, Connector_PinHeader_2.54mm:PinHeader_1x02_P2.54mm_Vertical, symbol Connector:Conn_01x02_Male
- removed J9: Powers, Connector_PinHeader_2.54mm:PinHeader_2x04_P2.54mm_Vertical, symbol Connector_Generic:Conn_02x04_Counter_Clockwise
- removed U1: ARDUINO_PRO_MINI, MODULE_ARDUINO_PRO_MINI, symbol Arduino pro mini:ARDUINO_PRO_MINI
- added A1: Arduino_Pro_Mini_Socket_NoSPH, PCM_arduino-library:Arduino_Pro_Mini_Socket_NoSPH, symbol PCM_arduino-library:Arduino_Pro_Mini_Socket_NoSPH
- added J13: Regulator-9v, Connector_PinHeader_2.54mm:PinHeader_2x02_P2.54mm_Vertical, symbol Connector:Conn_01x04_Male
- added J14: Input-Motor, Connector_PinHeader_2.54mm:PinHeader_1x02_P2.54mm_Vertical, symbol Connector:Conn_01x02_Male
- added J16: Button, Connector_PinHeader_2.54mm:PinHeader_2x02_P2.54mm_Vertical, symbol Connector:Conn_01x04_Male
- added J5: Regulator-5v, Connector_PinHeader_2.54mm:PinHeader_2x02_P2.54mm_Vertical, symbol Connector:Conn_01x04_Male
- added U1: DRV8833PW, Package_SO:TSSOP-16_4.4x5mm_P0.65mm, symbol Driver_Motor:DRV8833PW
- J3: value NRF-Power -> Input-Micro
- J7: value MOTOR-PWR-OUT -> Motor_Power
Connections:
- net +5V: now also A1.Vcc1 (Vcc), J5.3 (Pin_3); no longer J3.1 (Pin_1), J7.1 (Pin_1)
- net NRF_MISO: now reaches U2.7 (MISO)
- net NRF_MISO: now also A1.D12 (D12_MISO)
- net NRF_MOSI: now reaches U2.6 (MOSI)
- net NRF_MOSI: now also A1.D11 (D11_MOSI)
- net NRF_CSN: now reaches U2.4 (~{CSN})
- net NRF_CSN: now also A1.D10 (D10_CS)
- net NRF_SCK: now reaches U2.5 (SCK)
- net NRF_SCK: now also A1.D13 (D13_SCK)
- net PIN_SERVO: now reaches J2.3 (Pin_3)
- net PIN_SERVO: now also A1.D9
- net NRF_CE: now reaches U2.3 (CE)
- net NRF_CE: now also A1.D8
- net at J6.1 (Pin_1): now also U1.2 (AOUT1)
- net at J6.2 (Pin_2): now also U1.4 (AOUT2)
- net PIN_LED: now reaches J1.3 (Pin_3)
- net PIN_LED: now also A1.D7
- net PIN_ACCEL: now reaches J4.1 (Pin_1)
- net PIN_ACCEL: now also A1.D3 (D3_INT1)
- net PIN_HORN: now reaches J8.1 (Pin_1)
- net PIN_HORN: now also A1.D4
- net GND renamed GND2
- net GND2: now also A1.GND1 (GND), A1.GND2 (GND), J5.4 (Pin_4); no longer J3.2 (Pin_2), J7.2 (Pin_2)
- new net: J16.2 (Pin_2), J3.1 (Pin_1)
- new net: J3.2 (Pin_2), J5.2 (Pin_2)
- new net: J13.1 (Pin_1), J16.3 (Pin_3)
- new net: J13.2 (Pin_2), J14.2 (Pin_2)
- new net: J14.1 (Pin_1), J16.1 (Pin_1)
- new net: J16.4 (Pin_4), J5.1 (Pin_1)
- new net +9V: J13.3 (Pin_3), J7.1 (Pin_1), U1.11 (VCP)
- new net GND1: J13.4 (Pin_4), J7.2 (Pin_2), U1.13 (GND)
- new net PIN_MOTOR_1: A1.D5, U1.16 (AIN1)
- new net PIN_MOTOR_2: A1.D6, U1.15 (AIN2)
Other:
- moved on the sheet: J1, J2, J4, J6, J8

Commit message: schematic
Parts:
- removed A1: Arduino_Pro_Mini_Socket_NoSPH, PCM_arduino-library:Arduino_Pro_Mini_Socket_NoSPH, symbol PCM_arduino-library:Arduino_Pro_Mini_Socket_NoSPH
- removed J13: Regulator-9v, Connector_PinHeader_2.54mm:PinHeader_2x02_P2.54mm_Vertical, symbol Connector:Conn_01x04_Male
- removed J14: Input-Motor, Connector_PinHeader_2.54mm:PinHeader_1x02_P2.54mm_Vertical, symbol Connector:Conn_01x02_Male
- removed J16: Button, Connector_PinHeader_2.54mm:PinHeader_2x02_P2.54mm_Vertical, symbol Connector:Conn_01x04_Male
- removed J4: Accel, Connector_PinHeader_2.54mm:PinHeader_1x01_P2.54mm_Vertical, symbol Connector:Conn_01x01_Male
- added A3: Arduino_Pro_Mini_Socket_NoSPH, PCM_arduino-library:Arduino_Pro_Mini_Socket_NoSPH, symbol PCM_arduino-library:Arduino_Pro_Mini_Socket_NoSPH
- added J4: Power, Connector_PinHeader_2.54mm:PinHeader_1x02_P2.54mm_Vertical, symbol Connector:Conn_01x02_Male
- J3: value Input-Micro -> Battery
- J5: value Regulator-5v -> Switch
- J7: value Motor_Power -> BarGraph
Connections:
- net +5V: now also A3.Vcc1 (Vcc); no longer J5.3 (Pin_3)
- net NRF_CE: now also A3.D8
- net NRF_CSN: now also A3.D10 (D10_CS)
- net NRF_MISO: now also A3.D12 (D12_MISO)
- net NRF_MOSI: now also A3.D11 (D11_MOSI)
- net NRF_SCK: now also A3.D13 (D13_SCK)
- net PIN_HORN: now also A3.D4
- net PIN_LED: now also A3.D7
- net PIN_MOTOR_1: now also A3.D6
- net PIN_MOTOR_2: now also A3.D5
- net PIN_SERVO: now also A3.D9
- net -BATT: now reaches J3.1 (Pin_1)
- net -BATT: now also J7.1 (Pin_1)
- net +BATT: now reaches J3.2 (Pin_2), J5.2 (Pin_2)
- net +BATT: now also J5.4 (Pin_4), J7.2 (Pin_2)
- net +8V: now reaches J5.1 (Pin_1)
- net +8V: now also J5.3 (Pin_3), U1.11 (VCP), A3.RAW, J4.1 (Pin_1)
- removed net +9V: J7.1 (Pin_1), U1.11 (VCP)
- net GND1 renamed GND
- net GND: now also J1.1 (Pin_1), J2.1 (Pin_1), J8.2 (Pin_2), U2.1 (GND), A3.GND1 (GND), A3.GND2 (GND), J4.2 (Pin_2); no longer J7.2 (Pin_2)
- removed net GND2: J1.1 (Pin_1), J2.1 (Pin_1), J5.4 (Pin_4), J8.2 (Pin_2), U2.1 (GND)
Other:
- moved on the sheet: J5, U2

Commit message: Works
Parts:
- added J10: Reg-IN, Connector_PinHeader_2.54mm:PinHeader_1x02_P2.54mm_Vertical, symbol Connector:Conn_01x02_Male
- added J11: Reg-OUT, Connector_PinHeader_2.54mm:PinHeader_1x02_P2.54mm_Vertical, symbol Connector:Conn_01x02_Male
- added J12: Lamps, Connector_PinHeader_2.54mm:PinHeader_1x02_P2.54mm_Vertical, symbol Connector:Conn_01x02_Male
- added J13: Extra, Connector_PinHeader_2.54mm:PinHeader_1x02_P2.54mm_Vertical, symbol Connector:Conn_01x02_Male
- added J9: Regulator, Connector_PinHeader_2.54mm:PinHeader_2x02_P2.54mm_Vertical, symbol Connector:Conn_01x04_Male
- added JP1: Jumper_2_Bridged, Connector_PinHeader_2.54mm:PinHeader_1x02_P2.54mm_Vertical, symbol Jumper:Jumper_2_Bridged
Connections:
- net +5V: now also J11.1 (Pin_1), J9.3 (Pin_3)
- net +8V: now also J10.1 (Pin_1), J9.1 (Pin_1), JP1.1 (A); no longer A3.RAW
- net GND: now also J10.2 (Pin_2), J11.2 (Pin_2), J12.2 (Pin_2), J13.2 (Pin_2), J9.2 (Pin_2), J9.4 (Pin_4)
- net PIN_MOTOR_1: now also A3.D5; no longer A3.D6
- net PIN_MOTOR_2: now also A3.D6; no longer A3.D5
- net EXTRA: now reaches A3.D2 (D2_INT0)
- net EXTRA: now also J13.1 (Pin_1)
- net LAMPS: now reaches A3.D3 (D3_INT1)
- net LAMPS: now also J12.1 (Pin_1)
- new net: A3.RAW, JP1.2 (B)
